File: eerste_versie/eerste_versie.sch (KiCad schematic (older format))
At the start: 12 parts, among them U1 ESP32-WROOM-32U, U2 AMS1117-3.3, X1 DG3XX-02-5.0

Commit message: schema opgekuisd
Parts:
- PWR1: symbol Switch_out:SW_DIP_x01_OUTPUT -> eerste_versie-rescue:SW_DIP_x01_OUTPUT-Switch_out
- U1: symbol ESP32-WROOM-32U:ESP32-WROOM-32U -> eerste_versie-rescue:ESP32-WROOM-32U-ESP32-WROOM-32U
- X1: symbol degson:DG3XX-02-5.0 -> eerste_versie-rescue:DG3XX-02-5.0-degson
Other:
- note added: "ESP32"
- note added: "Voeding"
- moved on the sheet: BOOT1, C1, C2, C3, C4, EN1, Programmer_Header1, R1, U2

Commit message: tweede versie
Parts:
- added R2: 10k, Resistor_SMD:R_0805_2012Metric_Pad1.20x1.40mm_HandSolder, symbol Device:R
- C1, C2: footprint Capacitor_SMD:CP_Elec_6.3x3 -> Capacitor_SMD:C_0805_2012Metric_Pad1.18x1.45mm_HandSolder
- C4: value 47u -> 1u; footprint Capacitor_SMD:CP_Elec_6.3x3 -> Capacitor_SMD:C_0805_2012Metric_Pad1.18x1.45mm_HandSolder
Connections:
- net VDD33: now also R2.1
- net at BOOT1.1, U1.25 (IO0): now also R2.2
Other:
- moved on the sheet: BOOT1
Changed lines of the file:
@@
 F 0 "C2" H 1615 1496 50  0000 L CNN
 F 1 "100n" H 1615 1405 50  0000 L CNN
-F 2 "Capacitor_SMD:CP_Elec_6.3x3" H 1538 1300 50  0001 C CNN
+F 2 "Capacitor_SMD:C_0805_2012Metric_Pad1.18x1.45mm_HandSolder" H 1538 1300 50  0001 C CNN
 F 3 "~" H 1500 1450 50  0001 C CNN
 	1    1500 1450
@@
 P 6050 2250
 F 0 "C4" H 6165 2296 50  0000 L CNN
-F 1 "47u" H 6165 2205 50  0000 L CNN
-F 2 "Capacitor_SMD:CP_Elec_6.3x3" H 6050 2250 50  0001 C CNN
+F 1 "1u" H 6165 2205 50  0000 L CNN
+F 2 "Capacitor_SMD:C_0805_2012Metric_Pad1.18x1.45mm_HandSolder" H 6050 2250 50  0001 C CNN
 F 3 "~" H 6050 2250 50  0001 C CNN
 	1    6050 2250
@@
 $EndComp
 Wire Wire Line
-	2950 2900 2950 3000
-Wire Wire Line
-	3050 2900 2950 2900
+	2850 2900 2850 3000
+Wire Wire Line
+	2950 2900 2850 2900
 $Comp
 L power:GND #PWR04
 U 1 1 60453368
-P 2950 3000
-F 0 "#PWR04" H 2950 2750 50  0001 C CNN
-F 1 "GND" H 2955 2827 50  0000 C CNN
-F 2 "" H 2950 3000 50  0001 C CNN
-F 3 "" H 2950 3000 50  0001 C CNN
-	1    2950 3000
-	1    0    0    -1
-$EndComp
-Wire Wire Line
-	3800 2900 3650 2900
+P 2850 3000
+F 0 "#PWR04" H 2850 2750 50  0001 C CNN
+F 1 "GND" H 2855 2827 50  0000 C CNN
+F 2 "" H 2850 3000 50  0001 C CNN
+F 3 "" H 2850 3000 50  0001 C CNN
+	1    2850 3000
+	1    0    0    -1
+$EndComp
 $Comp
 L Switch:SW_DIP_x01 BOOT1
 U 1 1 60452495
-P 3350 2900
-F 0 "BOOT1" H 3350 2633 50  0000 C CNN
-F 1 "SW_DIP_x01" H 3350 2724 50  0000 C CNN
-F 2 "Button_Switch_SMD:SW_SPST_B3U-1000P" H 3350 2900 50  0001 C CNN
-F 3 "~" H 3350 2900 50  0001 C CNN
-	1    3350 2900
+P 3250 2900
+F 0 "BOOT1" H 3250 2633 50  0000 C CNN
+F 1 "SW_DIP_x01" H 3250 2724 50  0000 C CNN
+F 2 "Button_Switch_SMD:SW_SPST_B3U-1000P" H 3250 2900 50  0001 C CNN
+F 3 "~" H 3250 2900 50  0001 C CNN
+	1    3250 2900
 	-1   0    0    1
 $EndComp
@@
 F 0 "C1" V 5298 1400 50  0000 C CNN
 F 1 "100n" V 5389 1400 50  0000 C CNN
-F 2 "Capacitor_SMD:CP_Elec_6.3x3" H 5588 1250 50  0001 C CNN
+F 2 "Capacitor_SMD:C_0805_2012Metric_Pad1.18x1.45mm_HandSolder" H 5588 1250 50  0001 C CNN
 F 3 "~" H 5550 1400 50  0001 C CNN
 	1    5550 1400
@@
 Text Notes 3050 750  0    79   ~ 0
 ESP32
+$Comp
+L Device:R R2
+U 1 1 60511A7D
+P 3550 2550
+F 0 "R2" H 3620 2596 50  0000 L CNN
+F 1 "10k" H 3620 2505 50  0000 L CNN
+F 2 "Resistor_SMD:R_0805_2012Metric_Pad1.20x1.40mm_HandSolder" V 3480 2550 50  0001 C CNN
+F 3 "~" H 3550 2550 50  0001 C CNN
+	1    3550 2550
+	1    0    0    -1
+$EndComp
+Wire Wire Line
+	3550 2700 3550 2900
+Text GLabel 3550 2250 1    50   Input ~ 0
+VDD33
+Wire Wire Line
+	3550 2250 3550 2400
+Wire Wire Line
+	3550 2900 3800 2900
+Connection ~ 3550 2900
 $EndSCHEMATC

Commit message: update
Parts:
- added BZ1: Buzzer, CPT-1255C-090:CUI_CPT-1255C-090, symbol Device:Buzzer
- added D1: LED, LED_SMD:LED_0805_2012Metric_Pad1.15x1.40mm_HandSolder, symbol Device:LED
- added R3: TBD, Resistor_SMD:R_0805_2012Metric_Pad1.20x1.40mm_HandSolder, symbol Device:R
Connections:
- net GND: now also BZ1.2 (+), D1.1 (K)
- net at U1.14 (IO12): now also BZ1.1 (-)
- net at U1.16 (IO13): now also R3.2
- new net: D1.2 (A), R3.1
- no-connect marks 29 -> 27
Other:
- moved on the sheet: BOOT1, R2
Changed lines of the file:
@@
 	1    0    0    -1
-$EndComp
-Wire Wire Line
-	2850 2900 2850 3000
-Wire Wire Line
-	2950 2900 2850 2900
-$Comp
-L power:GND #PWR04
-U 1 1 60453368
-P 2850 3000
-F 0 "#PWR04" H 2850 2750 50  0001 C CNN
-F 1 "GND" H 2855 2827 50  0000 C CNN
-F 2 "" H 2850 3000 50  0001 C CNN
-F 3 "" H 2850 3000 50  0001 C CNN
-	1    2850 3000
-	1    0    0    -1
-$EndComp
-$Comp
-L Switch:SW_DIP_x01 BOOT1
-U 1 1 60452495
-P 3250 2900
-F 0 "BOOT1" H 3250 2633 50  0000 C CNN
-F 1 "SW_DIP_x01" H 3250 2724 50  0000 C CNN
-F 2 "Button_Switch_SMD:SW_SPST_B3U-1000P" H 3250 2900 50  0001 C CNN
-F 3 "~" H 3250 2900 50  0001 C CNN
-	1    3250 2900
-	-1   0    0    1
 $EndComp
 Connection ~ 5400 1400
@@
 NoConn ~ 3800 2800
 NoConn ~ 3800 2700
-NoConn ~ 3800 2600
-NoConn ~ 3800 2500
 NoConn ~ 3800 2400
 NoConn ~ 3800 2300
@@
 Text Notes 3050 750  0    79   ~ 0
 ESP32
+Wire Wire Line
+	2800 3400 2800 3500
+Wire Wire Line
+	2900 3400 2800 3400
+$Comp
+L power:GND #PWR04
+U 1 1 60453368
+P 2800 3500
+F 0 "#PWR04" H 2800 3250 50  0001 C CNN
+F 1 "GND" H 2805 3327 50  0000 C CNN
+F 2 "" H 2800 3500 50  0001 C CNN
+F 3 "" H 2800 3500 50  0001 C CNN
+	1    2800 3500
+	1    0    0    -1
+$EndComp
 $Comp
 L Device:R R2
 U 1 1 60511A7D
-P 3550 2550
-F 0 "R2" H 3620 2596 50  0000 L CNN
-F 1 "10k" H 3620 2505 50  0000 L CNN
-F 2 "Resistor_SMD:R_0805_2012Metric_Pad1.20x1.40mm_HandSolder" V 3480 2550 50  0001 C CNN
-F 3 "~" H 3550 2550 50  0001 C CNN
-	1    3550 2550
-	1    0    0    -1
-$EndComp
-Wire Wire Line
-	3550 2700 3550 2900
-Text GLabel 3550 2250 1    50   Input ~ 0
+P 3500 3750
+F 0 "R2" H 3570 3796 50  0000 L CNN
+F 1 "10k" H 3570 3705 50  0000 L CNN
+F 2 "Resistor_SMD:R_0805_2012Metric_Pad1.20x1.40mm_HandSolder" V 3430 3750 50  0001 C CNN
+F 3 "~" H 3500 3750 50  0001 C CNN
+	1    3500 3750
+	-1   0    0    1
+$EndComp
+Wire Wire Line
+	3500 3600 3500 3400
+Text GLabel 3500 4050 0    50   Input ~ 0
 VDD33
 Wire Wire Line
-	3550 2250 3550 2400
-Wire Wire Line
-	3550 2900 3800 2900
-Connection ~ 3550 2900
+	3500 4050 3500 3900
+Wire Wire Line
+	3500 3400 3750 3400
+Connection ~ 3500 3400
+$Comp
+L Switch:SW_DIP_x01 BOOT1
+U 1 1 60452495
+P 3200 3400
+F 0 "BOOT1" H 3200 3133 50  0000 C CNN
+F 1 "SW_DIP_x01" H 3200 3224 50  0000 C CNN
+F 2 "Button_Switch_SMD:SW_SPST_B3U-1000P" H 3200 3400 50  0001 C CNN
+F 3 "~" H 3200 3400 50  0001 C CNN
+	1    3200 3400
+	-1   0    0    1
+$EndComp
+$Comp
+L Device:Buzzer BZ1
+U 1 1 6052D7F8
+P 2900 2600
+F 0 "BZ1" H 2905 2890 50  0000 C CNN
+F 1 "Buzzer" H 2905 2799 50  0000 C CNN
+F 2 "CPT-1255C-090:CUI_CPT-1255C-090" V 2875 2700 50  0001 C CNN
+F 3 "~" V 2875 2700 50  0001 C CNN
+	1    2900 2600
+	-1   0    0    -1
+$EndComp
+Wire Wire Line
+	3000 2500 3800 2500
+Wire Wire Line
+	2950 3400 2900 3400
+Connection ~ 2900 3400
+$Comp
+L Device:R R3
+U 1 1 6053C92B
+P 3550 2750
+F 0 "R3" H 3480 2704 50  0000 R CNN
+F 1 "TBD" H 3480 2795 50  0000 R CNN
+F 2 "Resistor_SMD:R_0805_2012Metric_Pad1.20x1.40mm_HandSolder" V 3480 2750 50  0001 C CNN
+F 3 "~" H 3550 2750 50  0001 C CNN
+	1    3550 2750
+	-1   0    0    1
+$EndComp
+$Comp
+L Device:LED D1
+U 1 1 6053D592
+P 3550 3050
+F 0 "D1" V 3600 3200 50  0000 R CNN
+F 1 "LED" V 3500 3250 50  0000 R CNN
+F 2 "LED_SMD:LED_0805_2012Metric_Pad1.15x1.40mm_HandSolder" H 3550 3050 50  0001 C CNN
+F 3 "~" H 3550 3050 50  0001 C CNN
+	1    3550 3050
+	0    -1   -1   0
+$EndComp
+Wire Wire Line
+	3800 2600 3550 2600
+$Comp
+L power:GND #PWR09
+U 1 1 6053EC09
+P 3550 3200
+F 0 "#PWR09" H 3550 2950 50  0001 C CNN
+F 1 "GND" H 3550 3050 50  0000 C CNN
+F 2 "" H 3550 3200 50  0001 C CNN
+F 3 "" H 3550 3200 50  0001 C CNN
+	1    3550 3200
+	1    0    0    -1
+$EndComp
+Wire Wire Line
+	3800 2900 3750 2900
+Wire Wire Line
+	3750 2900 3750 3400
+$Comp
+L power:GND #PWR08
+U 1 1 60540F03
+P 3000 2750
+F 0 "#PWR08" H 3000 2500 50  0001 C CNN
+F 1 "GND" H 3005 2577 50  0000 C CNN
+F 2 "" H 3000 2750 50  0001 C CNN
+F 3 "" H 3000 2750 50  0001 C CNN
+	1    3000 2750
+	1    0    0    -1
+$EndComp
+Wire Wire Line
+	3000 2700 3000 2750
 $EndSCHEMATC

Commit message: derde_versie
Connections:
- net at U1.34 (RXD0): now also Programmer_Header1.2 (Pin_2); no longer Programmer_Header1.3 (Pin_3)
- net at U1.35 (TXD0): now also Programmer_Header1.3 (Pin_3); no longer Programmer_Header1.2 (Pin_2)
Other:
- moved on the sheet: Programmer_Header1
Changed lines of the file:
@@
 	1    0    0    -1
 $EndComp
-Wire Wire Line
-	5400 3300 5700 3300
-Wire Wire Line
-	5400 3400 5700 3400
 $Comp
 L power:GND #PWR05
@@
 	1    0    0    -1
 $EndComp
-Wire Wire Line
-	5700 3500 5700 3600
-$Comp
-L power:GND #PWR02
-U 1 1 60440D60
-P 5700 3600
-F 0 "#PWR02" H 5700 3350 50  0001 C CNN
-F 1 "GND" H 5705 3427 50  0000 C CNN
-F 2 "" H 5700 3600 50  0001 C CNN
-F 3 "" H 5700 3600 50  0001 C CNN
-	1    5700 3600
-	1    0    0    -1
-$EndComp
-Text GLabel 5700 3200 0    50   Input ~ 0
+Text GLabel 5800 3500 0    50   Input ~ 0
 VDD33
 Wire Wire Line
@@
 F 3 "" H 5500 3850 50  0001 C CNN
 	1    5500 3850
-	1    0    0    -1
-$EndComp
-$Comp
-L Connector_Generic:Conn_01x04 Programmer_Header1
-U 1 1 60440B4B
-P 5900 3300
-F 0 "Programmer_Header1" H 5980 3292 50  0000 L CNN
-F 1 "Conn_01x04" H 5980 3201 50  0000 L CNN
-F 2 "Connector_PinHeader_2.00mm:PinHeader_1x04_P2.00mm_Vertical" H 5900 3300 50  0001 C CNN
-F 3 "~" H 5900 3300 50  0001 C CNN
-	1    5900 3300
 	1    0    0    -1
 $EndComp
@@
 Wire Wire Line
 	3000 2700 3000 2750
+$Comp
+L Connector_Generic:Conn_01x04 Programmer_Header1
+U 1 1 60440B4B
+P 6000 3400
+F 0 "Programmer_Header1" H 6200 3550 50  0000 L CNN
+F 1 "Conn_01x04" H 6150 3350 50  0000 L CNN
+F 2 "Connector_PinHeader_2.00mm:PinHeader_1x04_P2.00mm_Vertical" H 6000 3400 50  0001 C CNN
+F 3 "~" H 6000 3400 50  0001 C CNN
+	1    6000 3400
+	1    0    0    1
+$EndComp
+Wire Wire Line
+	5800 3400 5400 3400
+Wire Wire Line
+	5800 3300 5400 3300
+Wire Wire Line
+	5800 3200 5750 3200
+$Comp
+L power:GND #PWR?
+U 1 1 6056E1B0
+P 5750 3200
+F 0 "#PWR?" H 5750 2950 50  0001 C CNN
+F 1 "GND" H 5650 3200 50  0000 C CNN
+F 2 "" H 5750 3200 50  0001 C CNN
+F 3 "" H 5750 3200 50  0001 C CNN
+	1    5750 3200
+	1    0    0    -1
+$EndComp
 $EndSCHEMATC

Commit message: volledige versie
Parts:
- removed C3: 47u, Capacitor_SMD:CP_Elec_6.3x3, symbol Device:CP1
- removed X1: DG3XX-02-5.0, degson:degson-DG306-5.0-02P, symbol eerste_versie-rescue:DG3XX-02-5.0-degson
- added C3: 10uF, Capacitor_SMD:C_0805_2012Metric_Pad1.18x1.45mm_HandSolder, symbol Device:C
- added C5: 100n, Capacitor_SMD:C_0805_2012Metric_Pad1.18x1.45mm_HandSolder, symbol Device:C
- added J1: 105017-1001, 105017-1001:MOLEX_105017-1001, symbol 105017-1001:105017-1001
- BOOT1, EN1: footprint Button_Switch_SMD:SW_SPST_B3U-1000P -> 434111043826:434111043826
- C2: value 100n -> 10uF
- PWR1: footprint Button_Switch_SMD:SW_DIP_SPSTx01_Slide_6.7x4.1mm_W6.73mm_P2.54mm_LowProfile_JPin -> sparkfun:SWITCH_SPST_SMD_A
- Prog_head: renamed from Programmer_Header1; footprint Connector_PinHeader_2.00mm:PinHeader_1x04_P2.00mm_Vertical -> Connector_PinHeader_2.54mm:PinHeader_1x04_P2.54mm_Vertical
Connections:
- net GND: now also C3.2, C5.1, J1.5, J1.S1 (SHIELD), J1.S2 (SHIELD), J1.S3 (SHIELD), J1.S4 (SHIELD), J1.S5 (SHIELD), J1.S6 (SHIELD)
- net VDD33: now also C3.1, C5.2
- net at U1.14 (IO12): no longer BZ1.1 (-)
- net at U1.23 (IO15): now also BZ1.1 (-)
- net at PWR1.1: now also J1.1
- no-connect marks 27 -> 30
Other:
- moved on the sheet: BOOT1, BZ1, C1, C2, C4, D1, EN1, PWR1, Prog_head, R1, R2, R3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

Commit message: nog een kleine aanpassing
Parts:
- renumbered Prog_head to Prog_head1
Changed lines of the file:
@@
 	2900 900  2900 800
 $Comp
-L Connector_Generic:Conn_01x04 Prog_head
+L Connector_Generic:Conn_01x04 Prog_head1
 U 1 1 60440B4B
 P 7650 4200
-F 0 "Prog_head" H 7850 4350 50  0000 L CNN
+F 0 "Prog_head1" H 7850 4350 50  0000 L CNN
 F 1 "Conn_01x04" H 7800 4150 50  0000 L CNN
 F 2 "Connector_PinHeader_2.54mm:PinHeader_1x04_P2.54mm_Vertical" H 7650 4200 50  0001 C CNN

Commit message: om te printen
Parts:
- Prog_head1: footprint Connector_PinHeader_2.54mm:PinHeader_1x04_P2.54mm_Vertical -> Connector_PinSocket_2.54mm:PinSocket_1x04_P2.54mm_Vertical
Changed lines of the file:
@@
 F 0 "Prog_head1" H 7850 4350 50  0000 L CNN
 F 1 "Conn_01x04" H 7800 4150 50  0000 L CNN
-F 2 "Connector_PinHeader_2.54mm:PinHeader_1x04_P2.54mm_Vertical" H 7650 4200 50  0001 C CNN
+F 2 "Connector_PinSocket_2.54mm:PinSocket_1x04_P2.54mm_Vertical" H 7650 4200 50  0001 C CNN
 F 3 "~" H 7650 4200 50  0001 C CNN
 	1    7650 4200
